File: Doc/PCB/Main_Board_v1/Controller.sch (KiCad schematic (older format))
At the start: 67 parts, among them J10 BPM, J11 UART, J12 I2C Interface LCD_C, J13 BUZZER_C, J16 IP, J17 -, J18 BREATH, J19 EP, J20 +, J21 VOL_MIN, J22 VOL, J23 VOL_MAX, J24 Conn_01x08, J25 POWEROFF, J26 PMAX, J7 TE_3.5mm_Screwless_P2, J8 SV2, J9 SV3, Q2 STP24NF10, Q3 STP24NF10, Q5 2N3904, U4 LM7805_TO220, U5 XPRESS-40, U6 LCD

Commit message: New V1 placement done. Speed up Monitor to 64 MHz
Parts:
- added RV2: 1K, Ventilator:Potentiometer_409HA, symbol Device:R_POT
Connections:
- net labels added: LD4, LD5, LD6, LD7, LDE, LDRS
- wire segments 314 -> 327
- no-connect marks 15 -> 12
Changed lines of the file:
@@
 Wire Wire Line
 	7250 4750 7300 4750
-NoConn ~ 5500 2450
-NoConn ~ 5500 3450
 Wire Wire Line
 	6650 2750 6950 2750
@@
 Wire Wire Line
 	9400 1900 9400 2050
-NoConn ~ 5500 3050
-NoConn ~ 5500 3150
 $Comp
 L Ventilator:XPRESS-40 U5
@@
 	8950 1400 9650 1400
 NoConn ~ 6650 2250
-NoConn ~ 6650 2350
-NoConn ~ 6650 2450
 NoConn ~ 6650 2550
 $Comp
@@
 	5100 6300 5100 5900
 Wire Wire Line
-	5200 5900 5200 6850
+	5200 5900 5200 6750
 Wire Wire Line
 	5300 5900 5300 6350
@@
 	4200 5900 4200 6050
 Wire Wire Line
-	4200 6050 5500 6050
+	4200 6050 4850 6050
 Connection ~ 5500 6050
 Wire Wire Line
@@
 Wire Wire Line
 	3150 5800 3150 6150
+$Comp
+L Device:R_POT RV?
+U 1 1 5EAE7B7C
+P 4850 6550
+AR Path="/5E9337AC/5EAE7B7C" Ref="RV?"  Part="1"
+AR Path="/5E9339D0/5EAE7B7C" Ref="RV2"  Part="1"
+F 0 "RV2" H 4780 6596 50  0000 R CNN
+F 1 "1K" H 4780 6505 50  0000 R CNN
+F 2 "Ventilator:Potentiometer_409HA" H 4850 6550 50  0001 C CNN
+F 3 "https://es.rs-online.com/web/p/resistencias-variables/6524546/" H 4850 6550 50  0001 C CNN
+	1    4850 6550
+	1    0    0    -1
+$EndComp
+Wire Wire Line
+	4850 6700 4850 6750
+Wire Wire Line
+	5000 6550 5400 6550
+Wire Wire Line
+	5400 6550 5400 5900
+Text Label 3950 6100 0    50   ~ 0
+LD7
+Text Label 3900 6150 0    50   ~ 0
+LD6
+Text Label 3800 6200 0    50   ~ 0
+LD5
+Text Label 3700 6250 0    50   ~ 0
+LD4
+Text Label 3900 6300 0    50   ~ 0
+LDE
+Text Label 3650 6350 0    50   ~ 0
+LDRS
+Wire Wire Line
+	4950 2350 5500 2350
+Wire Wire Line
+	5500 2450 4950 2450
+Wire Wire Line
+	5500 2050 4950 2050
+Wire Wire Line
+	5500 1950 4950 1950
+Wire Wire Line
+	5500 3050 5050 3050
+Wire Wire Line
+	5500 3150 5050 3150
+Text Label 5100 1950 0    50   ~ 0
+LD7
+Text Label 5100 2050 0    50   ~ 0
+LD6
+Text Label 5100 2350 0    50   ~ 0
+LD5
+Text Label 5100 2450 0    50   ~ 0
+LD4
+Text Label 5100 3050 0    50   ~ 0
+LDE
+Text Label 5100 3150 0    50   ~ 0
+LDRS
+NoConn ~ 6650 2050
+NoConn ~ 6650 2150
+NoConn ~ 5500 3550
+Wire Wire Line
+	4850 6750 5200 6750
+Connection ~ 5200 6750
+Wire Wire Line
+	5200 6750 5200 6850
+Wire Wire Line
+	4850 6400 4850 6050
+Connection ~ 4850 6050
+Wire Wire Line
+	4850 6050 5500 6050
 $EndSCHEMATC

Commit message: Version 1 of THT PCB
Parts:
- Q5: footprint Package_TO_SOT_THT:TO-92_Inline -> Ventilator:TO-92_Inline_Ventilator
Changed lines of the file:
@@
 F 0 "Q5" H 4190 7246 50  0000 L CNN
 F 1 "2N3904" H 4190 7155 50  0000 L CNN
-F 2 "Package_TO_SOT_THT:TO-92_Inline" H 4200 7125 50  0001 L CIN
+F 2 "Ventilator:TO-92_Inline_Ventilator" H 4200 7125 50  0001 L CIN
 F 3 "https://es.rs-online.com/web/p/transistores-bipolares-y-bjt/8051056/" H 4000 7200 50  0001 L CNN
 	1    4000 7200
@@
 	5500 3150 5050 3150
 Text Label 5100 1950 0    50   ~ 0
+LD4
+Text Label 5100 2050 0    50   ~ 0
+LD5
+Text Label 5100 2350 0    50   ~ 0
+LD6
+Text Label 5100 2450 0    50   ~ 0
 LD7
-Text Label 5100 2050 0    50   ~ 0
-LD6
-Text Label 5100 2350 0    50   ~ 0
-LD5
-Text Label 5100 2450 0    50   ~ 0
-LD4
 Text Label 5100 3050 0    50   ~ 0
 LDE

Commit message: Updated PCB
Parts:
- J25: footprint Ventilator:PushButton -> Ventilator:PH_2_pol
- R41, R42: value 460 -> 470
Changed lines of the file:
@@
 F 0 "J25" H 3278 3546 50  0000 L CNN
 F 1 "POWEROFF" H 3278 3455 50  0000 L CNN
-F 2 "Ventilator:PushButton" H 2950 3500 50  0001 C CNN
+F 2 "Ventilator:PH_2_pol" H 2950 3500 50  0001 C CNN
 F 3 "https://es.rs-online.com/web/p/botones-pulsadores/7346827/" H 2950 3500 50  0001 C CNN
 	1    2950 3500
@@
 AR Path="/5E9339D0/5F019076" Ref="R41"  Part="1"
 F 0 "R41" H 3220 6346 50  0000 L CNN
-F 1 "460" H 3220 6255 50  0000 L CNN
+F 1 "470" H 3220 6255 50  0000 L CNN
 F 2 "Resistor_THT:R_Axial_DIN0207_L6.3mm_D2.5mm_P10.16mm_Horizontal" V 3080 6300 50  0001 C CNN
 F 3 "~" H 3150 6300 50  0001 C CNN
@@
 AR Path="/5E9339D0/5F01907C" Ref="R42"  Part="1"
 F 0 "R42" H 3620 7246 50  0000 L CNN
-F 1 "460" H 3620 7155 50  0000 L CNN
+F 1 "470" H 3620 7155 50  0000 L CNN
 F 2 "Resistor_THT:R_Axial_DIN0207_L6.3mm_D2.5mm_P10.16mm_Horizontal" V 3480 7200 50  0001 C CNN
 F 3 "~" H 3550 7200 50  0001 C CNN
@@
 F 3 "https://es.rs-online.com/web/p/resistencias-variables/6524546/" H 4850 6550 50  0001 C CNN
 	1    4850 6550
-	1    0    0    -1
-$EndComp
-Wire Wire Line
+	1    0    0    1
+$EndComp
+Wire Wire Line
