File: Doc/PCB/Main_Board_v1/Main_Board_v1.kicad_pcb (KiCad board)
At the start: 2 copper layers, 83 parts, among them J1 TE_3.5mm_Screwless_P2, J10 PTR1, J11 UART, J12 I2C Interface LCD, J13 BUZZER_C, J2 TE_3.5mm_Screwless_P2, J3 UART_M, J4 Conn_01x08, J5 Buzzer, J6 I2C Interface LCD_M, J7 TE_3.5mm_Screwless_P2, J8 SP3, J9 SP2, Q1 IRLZ34N, Q2 IRLZ34N, Q3 IRLZ34N, U1 LM358, U2 LM7805_TO220, U3 XPRESS-40, U4 LM7805_TO220, U5 XPRESS-40

Commit message: First layout of Monitor
Parts:
- removed TP1: ALARM LED, Connector_PinHeader_2.54mm:PinHeader_1x02_P2.54mm_Vertical
- removed TP2: ALARM MUTE, Connector_PinHeader_2.54mm:PinHeader_1x02_P2.54mm_Vertical
- removed TP3: ALARM HISTORY, Connector_PinHeader_2.54mm:PinHeader_1x02_P2.54mm_Vertical
- added C21: 100nF, Capacitor_THT:C_Rect_L9.0mm_W3.3mm_P7.50mm_MKT, F.Cu at (58.3, 105.4)
- added J14: MUTE+LED, Ventilator:PH_4_pol, F.Cu at (152.4, 99.1)
- added J15: HISTORY, Ventilator:PH_2_pol, F.Cu at (152.4, 109.2)
- J5: value Buzzer -> BUZZER; footprint Connector_PinHeader_2.54mm:PinHeader_1x02_P2.54mm_Vertical -> Ventilator:PH_2_pol
- J6: footprint Connector_PinHeader_2.54mm:PinHeader_1x04_P2.54mm_Vertical -> Ventilator:PH_4_pol
- moved MK1 300.9 mm to (68.6, 127.0)
- moved D1 290.5 mm to (38.1, 63.5), turned to 90 degrees
- moved C20 240.6 mm to (86.4, 95.2), turned to 270 degrees
- moved R25 240.3 mm to (55.9, 83.8), turned to 270 degrees
- moved C18 239.1 mm to (405.0, 13.8)
- moved C19 239.1 mm to (334.0, 14.0)
- moved Q2 239.1 mm to (417.1, -4.79)
- moved Q3 239.1 mm to (417.1, -10.8)
- moved R13 239.1 mm to (391.5, 13.8)
- moved R16 239.1 mm to (424.1, -28.9)
- moved R19 239.1 mm to (424.1, -24.8)
- moved R20 239.1 mm to (410.7, -20.8)
- moved R21 239.1 mm to (424.1, -20.8)
- moved R22 239.1 mm to (410.7, -16.7)
- moved TP10 239.1 mm to (420.8, 4.42)
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Routing:
- net GND: track 75.8 -> 536.3 mm, vias 0 -> 1
- net +5V_M: track 18.2 -> 311.9 mm, vias 0 -> 2
- net SCL: track 0.00 -> 77.0 mm
- net SDA: track 0.00 -> 68.9 mm
- net /Monitor/MIC: track 0.00 -> 65.1 mm
- net /Monitor/MEAS_12V: track 0.00 -> 55.5 mm, vias 0 -> 1
- net +12V_M: track 39.9 -> 94.3 mm
- net /Monitor/SV1: track 0.00 -> 52.9 mm
- net /Monitor/nMCLR: track 0.00 -> 50.9 mm
- net /Monitor/ALARM_MUTE: track 0.00 -> 49.2 mm
- net /Monitor/ALARM_HISTORY: track 0.00 -> 47.0 mm
- net /Monitor/LCD_SCL_M: track 0.00 -> 45.5 mm
- net /Monitor/LCD_SDA_M: track 0.00 -> 45.5 mm
- net /Monitor/ICSPCLK_M: track 0.00 -> 43.5 mm
- net /Monitor/ICSPDAT_M: track 0.00 -> 40.6 mm
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
Commit message: Update in the PCB design. New docs and images
Parts:
- removed TP10: IP, Connector_PinHeader_2.54mm:PinHeader_1x02_P2.54mm_Vertical
- added C22: 1uF, Capacitor_THT:C_Rect_L7.0mm_W2.5mm_P5.00mm, F.Cu at (363.5, 81.4)
- added C23: 1uF, Capacitor_THT:C_Rect_L7.0mm_W2.5mm_P5.00mm, F.Cu at (359.6, 85.5)
- added C24: 1uF, Capacitor_THT:C_Rect_L7.0mm_W2.5mm_P5.00mm, F.Cu at (351.1, 85.5)
- added C25: 1uF, Capacitor_THT:C_Rect_L7.0mm_W2.5mm_P5.00mm, F.Cu at (342.5, 84.9)
- added C26: 1uF, Capacitor_THT:C_Rect_L7.0mm_W2.5mm_P5.00mm, F.Cu at (389.2, 63.1)
- added C27: 1uF, Capacitor_THT:C_Rect_L7.0mm_W2.5mm_P5.00mm, F.Cu at (355.0, 81.4)
- added C28: 100nF, Capacitor_THT:C_Rect_L9.0mm_W3.3mm_P7.50mm_MKT, F.Cu at (390.3, 39.7)
- added C29: 100nF, Capacitor_THT:C_Rect_L9.0mm_W3.3mm_P7.50mm_MKT, F.Cu at (368.9, 57.6)
- added C30: 100nF, Capacitor_THT:C_Rect_L9.0mm_W3.3mm_P7.50mm_MKT, F.Cu at (344.1, 80.5)
- added J16: IP, Ventilator:PushButton, F.Cu at (393.0, 54.5)
- added J17: -, Ventilator:PushButton, F.Cu at (357.8, 72.9)
- added J18: BREATH, Ventilator:PushButton_LED, B.Cu at (34.5, 70.4)
- added J19: EP, Ventilator:PushButton, F.Cu at (383.5, 48.6)
- added J20: +, Ventilator:PushButton, F.Cu at (402.2, 30.5)
- added J21: VOL_MIN, Ventilator:PushButton, F.Cu at (382.6, 58.1)
- added J22: VOL, Ventilator:PushButton, F.Cu at (367.3, 72.9)
- added J23: VOL_MAX, Ventilator:PushButton, F.Cu at (404.0, 40.0)
- added R26: 50, Resistor_THT:R_Axial_DIN0207_L6.3mm_D2.5mm_P10.16mm_Horizontal, F.Cu at (350.4, 63.1)
- added R27: 10k, Resistor_THT:R_Axial_DIN0207_L6.3mm_D2.5mm_P10.16mm_Horizontal, F.Cu at (375.2, 37.7)
- added R28: 10k, Resistor_THT:R_Axial_DIN0207_L6.3mm_D2.5mm_P10.16mm_Horizontal, F.Cu at (365.4, 47.2)
- added R29: 470, Resistor_THT:R_Axial_DIN0207_L6.3mm_D2.5mm_P10.16mm_Horizontal, F.Cu at (351.0, 57.6)
- added R30: 10k, Resistor_THT:R_Axial_DIN0207_L6.3mm_D2.5mm_P10.16mm_Horizontal, F.Cu at (375.2, 29.6)
- added R31: 10k, Resistor_THT:R_Axial_DIN0207_L6.3mm_D2.5mm_P10.16mm_Horizontal, F.Cu at (327.3, 71.4)
- added R32: 10k, Resistor_THT:R_Axial_DIN0207_L6.3mm_D2.5mm_P10.16mm_Horizontal, F.Cu at (317.5, 82.0)
- added S3: MPXV5004DP, Ventilator:1351-01, F.Cu at (146.3, 90.6)
- added S4: MPXV5004DP, Ventilator:1351-01, F.Cu at (217.4, 120.9)
- added TP1: TestPoint, Ventilator:LCD_DRILL, F.Cu at (48.0, 85.7)
- added TP2: TestPoint, Ventilator:LCD_DRILL, F.Cu at (123.1, 85.7)
- added TP3: TestPoint, Ventilator:LCD_DRILL, F.Cu at (47.9, 116.7)
- C17: value 1uF -> 100nF; footprint Capacitor_THT:C_Rect_L7.0mm_W2.5mm_P5.00mm -> Capacitor_THT:C_Rect_L9.0mm_W3.3mm_P7.50mm_MKT
- J10: value PTR1 -> BPM; footprint Connector_PinHeader_2.54mm:PinHeader_1x03_P2.54mm_Vertical -> Ventilator:PushButton
- J14: value MUTE+LED -> Button_LED; footprint Ventilator:PH_4_pol -> Ventilator:PushButton_LED; moved to B.Cu
- J15: value HISTORY -> Button; footprint Ventilator:PH_2_pol -> Ventilator:PushButton; moved to B.Cu
- J8: value SP3 -> SV2; footprint Connector_PinHeader_2.54mm:PinHeader_1x02_P2.54mm_Vertical -> Ventilator:PinHeader_1x02_Screwless_3.5mm
- J9: value SP2 -> SV3; footprint Connector_PinHeader_2.54mm:PinHeader_1x02_P2.54mm_Vertical -> Ventilator:PinHeader_1x02_Screwless_3.5mm
- R13: value 50 -> 470
- R14: value R -> 50
- TP4: value LED Breath -> TestPoint; footprint Connector_PinHeader_2.54mm:PinHeader_1x02_P2.54mm_Vertical -> Ventilator:LCD_DRILL
- TP5: value Breath -> TestPoint; footprint Connector_PinHeader_2.54mm:PinHeader_1x02_P2.54mm_Vertical -> Ventilator:LCD_DRILL
- TP6: value + -> TestPoint; footprint Connector_PinHeader_2.54mm:PinHeader_1x02_P2.54mm_Vertical -> Ventilator:LCD_DRILL
- TP7: value - -> TestPoint; footprint Connector_PinHeader_2.54mm:PinHeader_1x02_P2.54mm_Vertical -> Ventilator:LCD_DRILL
- TP8: value BPM -> TestPoint; footprint Connector_PinHeader_2.54mm:PinHeader_1x02_P2.54mm_Vertical -> Ventilator:LCD_DRILL
- TP9: value EP -> TestPoint_Alt; footprint Connector_PinHeader_2.54mm:PinHeader_1x02_P2.54mm_Vertical -> Ventilator:pcb; moved to B.Cu
- moved TP6 386.5 mm to (48.0, 68.8)
- moved TP7 335.5 mm to (122.9, 37.7)
- moved TP8 326.5 mm to (123.1, 68.7)
- moved TP9 314.6 mm to (107.4, 64.9), turned to 270 degrees
- moved TP4 311.2 mm to (123.1, 116.7)
- moved Q2 220.9 mm to (219.4, 93.7), turned to 90 degrees
- moved Q3 216.6 mm to (219.4, 77.7), turned to 90 degrees
- moved C15 213.6 mm to (233.2, 116.7), turned to 180 degrees
- moved J7 208.7 mm to (227.4, 109.1), turned to 90 degrees
- moved C17 208.0 mm to (344.1, 75.6)
- moved C16 205.4 mm to (353.9, 67.5), turned to 0 degrees
- moved C14 204.1 mm to (388.5, 30.0), turned to 0 degrees
- moved U5 203.5 mm to (142.0, 119.2), turned to 90 degrees
- moved R15 194.9 mm to (317.5, 86.1)
- moved U4 190.9 mm to (194.8, 89.9), turned to 0 degrees
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Connections:
- net /Controller/+12V_C renamed +12V_C
- C16 pad 1: /Controller/+5V_C -> +5V_C
- C17 pad 1: /Controller/+5V_C -> +5V_C
- C18 pad 1: Net-(C18-Pad1) -> /Controller/PR2
- C19 pad 1: /Controller/+5V_C -> +5V_C
- D2 pad 2: Net-(D2-Pad2) -> Net-(C24-Pad2)
- D3 pad 2: Net-(D3-Pad2) -> Net-(C25-Pad2)
- J10 pad 1: /Controller/+5V_C -> Net-(J10-Pad1)
- J10 pad 2: Net-(C18-Pad1) -> GND
- J11 pad 1: Net-(J11-Pad1) -> GND
- J11 pad 2: GND -> Net-(J11-Pad2)
- J12 pad 2: /Controller/+5V_C -> +5V_C
- J14 pad 1: Net-(J14-Pad1) -> /Monitor/ALARM_MUTE
- J14 pad 3: /Monitor/ALARM_MUTE -> Net-(J14-Pad3)
- J8 pad 2: Net-(D3-Pad2) -> Net-(C24-Pad2)
- J9 pad 2: Net-(D2-Pad2) -> Net-(C25-Pad2)
- Q2 pad 2: Net-(D2-Pad2) -> Net-(C24-Pad2)
- Q3 pad 2: Net-(D3-Pad2) -> Net-(C25-Pad2)
- R12 pad 1: Net-(J14-Pad1) -> Net-(J14-Pad3)
- R13 pad 1: Net-(Q2-Pad1) -> /Controller/PR2
- R14 pad 1: Net-(Q3-Pad1) -> Net-(Q2-Pad1)
- R14 pad 2: Net-(R14-Pad2) -> /Controller/SV2
- R15 pad 1: /Controller/+5V_C -> +5V_C
- R16 pad 1: Net-(R16-Pad1) -> Net-(J18-Pad3)
- R17 pad 1: /Controller/+5V_C -> +5V_C
- R18 pad 1: /Controller/+5V_C -> +5V_C
- R19 pad 1: /Controller/+5V_C -> +5V_C
- R19 pad 2: Net-(R19-Pad2) -> Net-(J20-Pad1)
- R20 pad 1: /Controller/+5V_C -> +5V_C
- R20 pad 2: Net-(R20-Pad2) -> Net-(J16-Pad1)
- R21 pad 1: /Controller/+5V_C -> +5V_C
- R21 pad 2: Net-(R21-Pad2) -> Net-(J19-Pad1)
- R22 pad 1: /Controller/+5V_C -> +5V_C
- R22 pad 2: Net-(R22-Pad2) -> Net-(J10-Pad1)
- R23 pad 1: /Controller/+5V_C -> +5V_C
- R23 pad 2: Net-(R23-Pad2) -> Net-(J18-Pad2)
- TP4 pad 1: Net-(R16-Pad1) -> GND
- TP5 pad 1: Net-(R23-Pad2) -> GND
- TP6 pad 1: Net-(R22-Pad2) -> GND
- TP7 pad 1: Net-(R21-Pad2) -> GND
- TP8 pad 1: Net-(R20-Pad2) -> GND
- U4 pad 3: /Controller/+5V_C -> +5V_C
- U5 pad 11: /Controller/+5V_C -> +5V_C
- U5 pad 15: Net-(J11-Pad1) -> Net-(J11-Pad2)
- U5 pad 2: Net-(C18-Pad1) -> /Controller/PR2
- U5 pad 21: Net-(R19-Pad2) -> Net-(J20-Pad1)
- U5 pad 22: Net-(R20-Pad2) -> Net-(J16-Pad1)
- U5 pad 27: Net-(R21-Pad2) -> Net-(J19-Pad1)
- U5 pad 28: Net-(R22-Pad2) -> Net-(J10-Pad1)
- U5 pad 29: Net-(R23-Pad2) -> Net-(J18-Pad2)
- U5 pad 3: Net-(R13-Pad2) -> /Controller/SV2
- U5 pad 32: /Controller/+5V_C -> +5V_C
- U5 pad 4: Net-(R14-Pad2) -> /Controller/SV3
- U5 pad 5: Net-(U5-Pad5) -> /Controller/PR3
Routing:
- net GND: track 536.3 -> 0.00 mm, vias 1 -> 0
- net +5V_M: track 311.9 -> 0.00 mm, vias 2 -> 0
- net +12V_M: track 94.3 -> 0.00 mm
- net SCL: track 77.0 -> 0.00 mm
- net SDA: track 68.9 -> 0.00 mm
- net /Monitor/MIC: track 65.1 -> 0.00 mm
- net /Monitor/MEAS_12V: track 55.5 -> 0.00 mm, vias 1 -> 0
- net /Monitor/SV1: track 52.9 -> 0.00 mm
- net /Monitor/nMCLR: track 50.9 -> 0.00 mm
- net /Monitor/ALARM_MUTE: track 49.2 -> 0.00 mm
- net /Monitor/ALARM_HISTORY: track 47.0 -> 0.00 mm
- net /Monitor/LCD_SCL_M: track 45.5 -> 0.00 mm
- net /Monitor/LCD_SDA_M: track 45.5 -> 0.00 mm
- net /Monitor/ICSPCLK_M: track 43.5 -> 0.00 mm
- net /Monitor/ICSPDAT_M: track 40.6 -> 0.00 mm
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Other:
- board outline added: 211 x 98 mm
- net class Default: clearance 0.2 -> 0.4; trace_width 0.25 -> 0.35; via_dia 0.8 -> 0.9; via_drill 0.4 -> 0.6
- net class Power: clearance 0.2 -> 0.4; via_dia 0.8 -> 0.9; via_drill 0.4 -> 0.6
- rule trace_clearance: 0.2 -> 0.4

Commit message: First placement of board
Parts:
- added J24: Conn_01x08, Connector_PinHeader_2.54mm:PinHeader_1x08_P2.54mm_Horizontal, F.Cu at (148.2, 119.8)
- added R33: 470, Resistor_THT:R_Axial_DIN0207_L6.3mm_D2.5mm_P10.16mm_Horizontal, F.Cu at (94.3, 78.9)
- added R34: 470, Resistor_THT:R_Axial_DIN0207_L6.3mm_D2.5mm_P10.16mm_Horizontal, F.Cu at (94.5, 74.0)
- added R35: 10k, Resistor_THT:R_Axial_DIN0207_L6.3mm_D2.5mm_P10.16mm_Horizontal, F.Cu at (40.7, 65.6)
- added R36: 10k, Resistor_THT:R_Axial_DIN0207_L6.3mm_D2.5mm_P10.16mm_Horizontal, F.Cu at (153.3, 129.2)
- C1, C11, C12, C13, C14, C16, C17, C19, C21, C28, C29, C30, C7, C8, C9: value 100nF -> 100nF - 100V; footprint Capacitor_THT:C_Rect_L9.0mm_W3.3mm_P7.50mm_MKT -> Capacitor_THT:C_Rect_L7.2mm_W2.5mm_P5.00mm_FKS2_FKP2_MKS2_MKP2
- C10, C18, C2, C20, C22, C23, C24, C25, C26, C27, C3, C4, C6: footprint Capacitor_THT:C_Rect_L7.0mm_W2.5mm_P5.00mm -> Capacitor_THT:C_Rect_L13.0mm_W4.0mm_P10.00mm_FKS3_FKP3_MKS4
- C15, C5: footprint Capacitor_THT:CP_Radial_D5.0mm_P2.50mm -> Capacitor_THT:CP_Radial_D5.0mm_P2.00mm
- J10, J16, J17, J19, J20, J21, J22, J23, J6: moved to B.Cu
- J12: value I2C Interface LCD -> I2C Interface LCD_C; footprint Connector_PinHeader_2.54mm:PinHeader_1x04_P2.54mm_Vertical -> Ventilator:PH_4_pol; moved to B.Cu
- moved J20 369.9 mm to (38.5, 98.0)
- moved J23 349.3 mm to (56.5, 75.4), turned to 180 degrees
- moved J13 340.8 mm to (61.5, 87.5), turned to 270 degrees
- moved J16 323.9 mm to (76.5, 123.3), turned to 180 degrees
- moved J17 321.1 mm to (38.6, 107.4), turned to 180 degrees
- moved R16 320.3 mm to (32.4, 82.8)
- moved J22 312.8 mm to (58.5, 123.4), turned to 180 degrees
- moved J21 308.5 mm to (74.6, 75.4), turned to 180 degrees
- moved C28 307.9 mm to (85.8, 85.6), turned to 180 degrees
- moved R18 305.0 mm to (48.8, 94.8)
- moved R30 304.1 mm to (83.8, 116.8)
- moved R23 298.6 mm to (42.1, 79.2), turned to 90 degrees
- moved J19 298.6 mm to (94.5, 123.4), turned to 180 degrees
- moved R27 289.8 mm to (89.3, 85.6)
- moved R22 282.2 mm to (105.9, 118.2), turned to 270 degrees
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Connections:
- net /Monitor/nMCLR renamed /Monitor/nMCLR_M
- U5 pad 1: Net-(U5-Pad1) -> /Controller/nMCLR_C
- U5 pad 39: Net-(U5-Pad39) -> /Controller/ICSPCLK_C
- U5 pad 40: Net-(U5-Pad40) -> /Controller/ICSPDAT_C
Other:
- board size 211 x 98 mm -> 180 x 98 mm

Commit message: Update in PCB: Schematic and Layout
Parts:
- added TP10: TestPoint, Ventilator:LCD_DRILL, F.Cu at (188.4, 37.9)
- added TP11: TestPoint, Ventilator:LCD_DRILL, F.Cu at (188.4, 126.9)
- added TP12: TestPoint, Ventilator:LCD_DRILL, F.Cu at (32.4, 37.9)
- added TP13: TestPoint, Ventilator:LCD_DRILL, F.Cu at (32.4, 126.7)
- MK1: footprint Connector_PinHeader_2.54mm:PinHeader_1x02_P2.54mm_Vertical -> Ventilator:MIC
- moved C11 87.9 mm to (90.4, 66.9), turned to 0 degrees
- moved C20 80.2 mm to (82.0, 67.2), turned to 180 degrees
- moved C8 71.5 mm to (164.4, 48.9), turned to 0 degrees
- moved C15 55.5 mm to (184.4, 79.9)
- moved C16 43.7 mm to (172.4, 110.9)
- moved J5 41.6 mm to (99.4, 35.9)
- moved C14 38.4 mm to (172.4, 95.9), turned to 0 degrees
- moved R30 37.3 mm to (68.4, 82.9), turned to 90 degrees
- moved J7 37.2 mm to (176.4, 90.9)
- moved U4 35.3 mm to (171.0, 104.4), turned to 0 degrees
- moved R19 30.8 mm to (54.4, 98.9)
- moved MK1 24.3 mm to (62.9, 36.7), turned to 0 degrees
- moved C22 22.5 mm to (142.4, 96.5), turned to 180 degrees
- moved R4 21.7 mm to (57.4, 47.9), turned to 270 degrees
- moved R21 18.2 mm to (87.4, 128.9), turned to 90 degrees
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
Commit message: New PCB version; I2C Slave works
Parts:
- removed TP5, TP6, TP7, TP8: TestPoint, Ventilator:LCD_DRILL
- added J25: POWEROFF, Ventilator:PushButton, F.Cu at (93.4, 2.39)
- added J26: PMAX, Ventilator:PushButton, F.Cu at (80.1, 10.5)
- added R37: 10k, Resistor_THT:R_Axial_DIN0207_L6.3mm_D2.5mm_P10.16mm_Horizontal, F.Cu at (77.0, 1.49)
- added R38: 10k, Resistor_THT:R_Axial_DIN0207_L6.3mm_D2.5mm_P10.16mm_Horizontal, F.Cu at (77.0, 5.54)
- added U6: LCD, Ventilator:LCD_2x16, F.Cu at (-9.47, 65.9)
- J14: value Button_LED -> MUTE
- J15: value Button -> HISTORY
- Q1, Q2, Q3: value IRLZ34N -> STP24NF10
- R14, R26, R6: value 50 -> 1k
- R24: value 22k -> 2k2
- R25: value 10k -> 1k
- R27, R28: value 10k -> 2k2
- S2, S3: value MPXV5004DP -> MPXV5010DP
- moved S2 33.9 mm to (228.0, 46.8), turned to 0 degrees
- moved S3 0.34 mm to (195.0, 100.2)
Connections:
- net Net-(J11-Pad2) renamed /Controller/RX_C
- net Net-(J11-Pad3) renamed /Controller/TX_C
- C18 pad 1: /Controller/PR2 -> /Controller/PR_MAIN
- C27 pad 1: /Controller/PR3 -> /Controller/PR_AUX
- J12 pad 3: /Controller/LCD_SDA -> SDA
- J12 pad 4: /Controller/LCD_SCL -> SCL
- R13 pad 1: /Controller/PR2 -> /Controller/PR_MAIN
- R15 pad 2: /Controller/LCD_SCL -> SCL
- R17 pad 2: /Controller/LCD_SDA -> SDA
- R29 pad 1: /Controller/PR3 -> /Controller/PR_AUX
- U5 pad 10: Net-(U5-Pad10) -> /Controller/PR_AUX
- U5 pad 18: SCL -> Net-(U5-Pad18)
- U5 pad 2: /Controller/PR2 -> Net-(U5-Pad2)
- U5 pad 20: Net-(J17-Pad1) -> Net-(J16-Pad1)
- U5 pad 21: Net-(J20-Pad1) -> Net-(J19-Pad1)
- U5 pad 22: Net-(J16-Pad1) -> Net-(J10-Pad1)
- U5 pad 23: SDA -> Net-(J26-Pad1)
- U5 pad 27: Net-(J19-Pad1) -> Net-(J20-Pad1)
- U5 pad 28: Net-(J10-Pad1) -> Net-(J18-Pad2)
- U5 pad 29: Net-(J18-Pad2) -> Net-(R16-Pad2)
- U5 pad 3: /Controller/SV2 -> Net-(U5-Pad3)
- U5 pad 30: Net-(R16-Pad2) -> Net-(J17-Pad1)
- U5 pad 34: Net-(U5-Pad34) -> SCL
- U5 pad 35: Net-(U5-Pad35) -> SDA
- U5 pad 37: /Controller/LCD_SDA -> Net-(U5-Pad37)
- U5 pad 38: /Controller/LCD_SCL -> Net-(U5-Pad38)
- U5 pad 4: /Controller/SV3 -> /Controller/SV2
- U5 pad 5: /Controller/PR3 -> /Controller/SV3
- U5 pad 6: Net-(C26-Pad1) -> Net-(U5-Pad6)
- U5 pad 8: Net-(U5-Pad8) -> Net-(C26-Pad1)
- U5 pad 9: Net-(U5-Pad9) -> /Controller/PR_MAIN

Commit message: New V1 placement done. Speed up Monitor to 64 MHz
Parts:
- removed TP10, TP11, TP12, TP13: TestPoint, Ventilator:LCD_DRILL
- removed TP9: TestPoint_Alt, Ventilator:pcb
- added Q4: 2N3904, Package_TO_SOT_THT:TO-92_Inline, F.Cu at (119.9, 60.9)
- added Q5: 2N3904, Package_TO_SOT_THT:TO-92_Inline, F.Cu at (108.4, 106.9)
- added R39: 460, Resistor_THT:R_Axial_DIN0207_L6.3mm_D2.5mm_P10.16mm_Horizontal, F.Cu at (119.9, 54.9)
- added R40: 460, Resistor_THT:R_Axial_DIN0207_L6.3mm_D2.5mm_P10.16mm_Horizontal, F.Cu at (126.9, 50.9)
- added R41: 460, Resistor_THT:R_Axial_DIN0207_L6.3mm_D2.5mm_P10.16mm_Horizontal, F.Cu at (93.9, 89.4)
- added R42: 460, Resistor_THT:R_Axial_DIN0207_L6.3mm_D2.5mm_P10.16mm_Horizontal, F.Cu at (118.4, 90.9)
- added R43: 4.7, Resistor_THT:R_Axial_DIN0207_L6.3mm_D2.5mm_P10.16mm_Horizontal, F.Cu at (115.9, 104.9)
- added RV1: 1K, Ventilator:Potentiometer_409HA, F.Cu at (127.9, 68.9)
- added RV2: 1K, Ventilator:Potentiometer_409HA, F.Cu at (113.4, 90.9)
- added U7: LCD, Ventilator:LCD_2x16, F.Cu at (117.9, 36.4)
- J25: footprint Ventilator:PushButton -> Ventilator:PH_2_pol
- J26: moved to B.Cu
- moved U6 129.8 mm to (118.9, 85.4)
- moved R38 127.5 mm to (39.4, 127.4)
- moved J26 115.1 mm to (55.4, 122.9), turned to 180 degrees
- moved J25 114.6 mm to (47.4, 107.4)
- moved R37 94.2 mm to (48.9, 91.4), turned to 270 degrees
- moved TP4 88.7 mm to (189.9, 126.9)
- moved TP1 67.0 mm to (189.9, 36.9)
- moved U5 62.6 mm to (53.9, 111.4), turned to 90 degrees
- moved TP2 60.5 mm to (31.4, 126.9)
- moved J21 58.1 mm to (34.4, 117.4)
- moved C26 49.6 mm to (60.4, 82.9)
- moved R30 48.3 mm to (41.4, 122.9)
- moved R28 45.2 mm to (59.4, 77.9)
- moved J23 37.5 mm to (34.4, 105.7)
- moved J5 35.0 mm to (112.4, 68.4)
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Connections:
- J11 pad 2: /Controller/RX_C -> /Controller/TX_C
- J11 pad 3: /Controller/TX_C -> /Controller/RX_C
- U3 pad 19: Net-(U3-Pad19) -> /Monitor/BUZZER
- U3 pad 20: Net-(U3-Pad20) -> /Monitor/ALARM_HISTORY
- U3 pad 21: Net-(U3-Pad21) -> /Monitor/ALARM_MUTE
- U3 pad 22: Net-(U3-Pad22) -> /Monitor/ALARM_LED
- U3 pad 27: /Monitor/BUZZER -> Net-(U3-Pad27)
- U3 pad 28: /Monitor/ALARM_HISTORY -> Net-(U3-Pad28)
- U3 pad 29: /Monitor/ALARM_MUTE -> Net-(U3-Pad29)
- U3 pad 30: /Monitor/ALARM_LED -> Net-(U3-Pad30)
- U5 pad 13: Net-(U5-Pad13) -> /Controller/LDE
- U5 pad 14: Net-(U5-Pad14) -> /Controller/LDRS
- U5 pad 2: Net-(U5-Pad2) -> /Controller/LD7
- U5 pad 3: Net-(U5-Pad3) -> /Controller/LD6
- U5 pad 6: Net-(U5-Pad6) -> /Controller/LD5
- U5 pad 7: Net-(U5-Pad7) -> /Controller/LD4
- U6 pad 1: (no net) -> GND
- U6 pad 11: (no net) -> /Controller/LD4
- U6 pad 12: (no net) -> /Controller/LD5
- U6 pad 13: (no net) -> /Controller/LD6
- U6 pad 14: (no net) -> /Controller/LD7
- U6 pad 15: (no net) -> +5V_C
- U6 pad 16: (no net) -> Net-(R43-Pad1)
- U6 pad 2: (no net) -> +5V_C
- U6 pad 3: (no net) -> Net-(RV2-Pad2)
- U6 pad 4: (no net) -> /Controller/LDRS
- U6 pad 5: (no net) -> GND
- U6 pad 6: (no net) -> /Controller/LDE

Commit message: Version 1 of THT PCB
Parts:
- J25: footprint Ventilator:PH_2_pol -> Ventilator:PushButton
- Q4, Q5: footprint Package_TO_SOT_THT:TO-92_Inline -> Ventilator:TO-92_Inline_Ventilator
- RV1, RV2: moved to B.Cu
- moved R28 65.3 mm to (117.9, 106.9), turned to 270 degrees
- moved Q4 61.2 mm to (62.4, 39.9), turned to 90 degrees
- moved C26 53.8 mm to (109.9, 103.9), turned to 270 degrees
- moved U5 53.3 mm to (103.9, 92.9), turned to 270 degrees
- moved R40 48.3 mm to (79.9, 39.9), turned to 180 degrees
- moved R39 47.5 mm to (76.4, 35.9), turned to 180 degrees
- moved R27 42.2 mm to (114.4, 114.4), turned to 90 degrees
- moved R43 42.2 mm to (80.9, 81.4), turned to 0 degrees
- moved J3 41.8 mm to (102.4, 67.9), turned to 90 degrees
- moved R41 31.7 mm to (124.4, 80.9), turned to 180 degrees
- moved Q5 28.7 mm to (97.4, 80.4), turned to 180 degrees
- moved MK1 21.6 mm to (41.4, 36.4)
- moved R34 17.2 mm to (84.8, 73.8)
- moved R33 16.9 mm to (84.8, 76.8)
- moved R42 12.2 mm to (111.4, 80.9), turned to 180 degrees
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Connections:
- U5 pad 2: /Controller/LD7 -> /Controller/LD4
- U5 pad 3: /Controller/LD6 -> /Controller/LD5
- U5 pad 6: /Controller/LD5 -> /Controller/LD6
- U5 pad 7: /Controller/LD4 -> /Controller/LD7
Routing:
- net GND: track 0.00 -> 1273.2 mm, vias 0 -> 7
- net +5V_M: track 0.00 -> 434.1 mm, vias 0 -> 2
- net +5V_C: track 0.00 -> 412.7 mm
- net SCL: track 0.00 -> 180.6 mm, vias 0 -> 4
- net SDA: track 0.00 -> 177.2 mm, vias 0 -> 5
- net /Monitor/PTR4: track 0.00 -> 145.6 mm, vias 0 -> 1
- net /Controller/PR_AUX: track 0.00 -> 141.1 mm, vias 0 -> 1
- net /Monitor/PTR2: track 0.00 -> 136.0 mm
- net /Controller/PR_MAIN: track 0.00 -> 125.8 mm
- net /Monitor/MEAS_12V: track 0.00 -> 112.0 mm, vias 0 -> 1
- net +12V_C: track 0.00 -> 86.2 mm
- net /Monitor/SV1: track 0.00 -> 85.1 mm, vias 0 -> 1
- net +12V_M: track 0.00 -> 79.7 mm
- net Net-(J10-Pad1): track 0.00 -> 73.6 mm
- net /Controller/nMCLR_C: track 0.00 -> 66.7 mm, vias 0 -> 1
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
Commit message: Updated PCB
Parts:
- J25: footprint Ventilator:PushButton -> Ventilator:PH_2_pol
- R39, R40, R41, R42: value 460 -> 470
- RV1, RV2: moved to F.Cu
- moved RV2 5.04 mm to (112.3, 100.4)
- moved RV1 4.90 mm to (123.6, 55.5)
Connections:
- RV1 pad 1: +5V_M -> GND
- RV1 pad 3: GND -> +5V_M
- RV2 pad 1: +5V_C -> GND
- RV2 pad 3: GND -> +5V_C
