File: Doc/PCB/Main_Board_v1/Monitor.sch (KiCad schematic (older format))
At the start: 58 parts, among them J1 TE_3.5mm_Screwless_P2, J14 MUTE, J15 HISTORY, J2 TE_3.5mm_Screwless_P2, J3 UART_M, J4 Conn_01x08, J5 BUZZER, J6 I2C Interface LCD_M, Q1 STP24NF10, Q4 2N3904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

Commit message: Version 1 of THT PCB
Parts:
- Q4: footprint Package_TO_SOT_THT:TO-92_Inline -> Ventilator:TO-92_Inline_Ventilator
Changed lines of the file:
@@
 F 0 "Q4" H 8290 5746 50  0000 L CNN
 F 1 "2N3904" H 8290 5655 50  0000 L CNN
-F 2 "Package_TO_SOT_THT:TO-92_Inline" H 8300 5625 50  0001 L CIN
+F 2 "Ventilator:TO-92_Inline_Ventilator" H 8300 5625 50  0001 L CIN
 F 3 "https://es.rs-online.com/web/p/transistores-bipolares-y-bjt/8051056/" H 8100 5700 50  0001 L CNN
 	1    8100 5700

Commit message: Updated PCB
Parts:
- R39, R40: value 460 -> 470
Connections:
- net +5V_M: now also RV1.3; no longer RV1.1
- net GND: now also RV1.1; no longer RV1.3
Changed lines of the file:
@@
 AR Path="/5E9337AC/5EE73DD7" Ref="R39"  Part="1"
 F 0 "R39" H 7170 5346 50  0000 L CNN
-F 1 "460" H 7170 5255 50  0000 L CNN
+F 1 "470" H 7170 5255 50  0000 L CNN
 F 2 "Resistor_THT:R_Axial_DIN0207_L6.3mm_D2.5mm_P10.16mm_Horizontal" V 7030 5300 50  0001 C CNN
 F 3 "~" H 7100 5300 50  0001 C CNN
@@
 AR Path="/5E9337AC/5EE87117" Ref="R40"  Part="1"
 F 0 "R40" H 7720 5746 50  0000 L CNN
-F 1 "460" H 7720 5655 50  0000 L CNN
+F 1 "470" H 7720 5655 50  0000 L CNN
 F 2 "Resistor_THT:R_Axial_DIN0207_L6.3mm_D2.5mm_P10.16mm_Horizontal" V 7580 5700 50  0001 C CNN
 F 3 "~" H 7650 5700 50  0001 C CNN
@@
 F 3 "https://es.rs-online.com/web/p/resistencias-variables/6524546/" H 8950 5550 50  0001 C CNN
 	1    8950 5550
-	1    0    0    -1
+	1    0    0    1
 $EndComp
 Wire Wire Line
