File: Doc/PCB/Main_Board_v1_2/Main_Board_v1_2.kicad_pcb (KiCad board)
At the start: 2 copper layers, 180 x 98 mm, 131 parts, among them J1 SV1, J10 BPM, J11 UART, J12 I2C Interface LCD_C, J13 BUZZER_C, J14 MUTE, J15 HISTORY, J16 IP, J17 -, J18 BREATH, J19 EP, J2 +12V, J20 +, J21 VOL_MIN, J22 VOL, J23 VOL_MAX, J24 Conn_01x08, J25 POWEROFF, J26 PMAX, J27 SV2, J3 UART_M, J4 Conn_01x08, J5 BUZZER_M, J6 I2C Interface LCD_M, J7 +12V, J8 SV2, J9 SV3, Q1 STP24NF10, Q2 STP24NF10, Q3 STP24NF10, Q4 2N3904, Q5 2N3904, Q6 STP24NF10, U1 LM358, U2 LM7805_TO220, U3 XPRESS-40, U4 LM7805_TO220, U5 XPRESS-40, U6 LCD, U7 LCD

Commit message: Fixed SilkScreen V1.2 THT
Parts:
- J27: value SV2 -> SV4
- J5: value BUZZER_M -> BUZZER
Other:
- board text added: "FLOW"
- board text added: "PRESSEXT"
- board text added: "PRESS_INT"
Changed lines of the file:
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@@
   (general
     (thickness 1.6)
-    (drawings 25)
+    (drawings 29)
     (tracks 1418)
     (zones 0)
@@
     (add_net "Net-(J22-Pad1)")
     (add_net "Net-(J23-Pad1)")
+    (add_net "Net-(J24-Pad6)")
+    (add_net "Net-(J24-Pad7)")
+    (add_net "Net-(J24-Pad8)")
     (add_net "Net-(J25-Pad2)")
     (add_net "Net-(J26-Pad1)")
+    (add_net "Net-(J4-Pad6)")
+    (add_net "Net-(J4-Pad7)")
+    (add_net "Net-(J4-Pad8)")
     (add_net "Net-(Q1-Pad1)")
     (add_net "Net-(Q2-Pad1)")
@@
     (add_net "Net-(RV1-Pad2)")
     (add_net "Net-(RV2-Pad2)")
+    (add_net "Net-(S1-Pad1)")
+    (add_net "Net-(S1-Pad5)")
+    (add_net "Net-(S1-Pad6)")
+    (add_net "Net-(S1-Pad7)")
+    (add_net "Net-(S1-Pad8)")
+    (add_net "Net-(S2-Pad1)")
+    (add_net "Net-(S2-Pad5)")
+    (add_net "Net-(S2-Pad6)")
+    (add_net "Net-(S2-Pad7)")
+    (add_net "Net-(S2-Pad8)")
+    (add_net "Net-(S3-Pad1)")
+    (add_net "Net-(S3-Pad5)")
+    (add_net "Net-(S3-Pad6)")
+    (add_net "Net-(S3-Pad7)")
+    (add_net "Net-(S3-Pad8)")
+    (add_net "Net-(S4-Pad1)")
+    (add_net "Net-(S4-Pad5)")
+    (add_net "Net-(S4-Pad6)")
+    (add_net "Net-(S4-Pad7)")
+    (add_net "Net-(S4-Pad8)")
     (add_net "Net-(U3-Pad10)")
     (add_net "Net-(U3-Pad13)")
@@
     (add_net "Net-(U5-Pad36)")
     (add_net "Net-(U5-Pad37)")
+    (add_net "Net-(U6-Pad10)")
+    (add_net "Net-(U6-Pad7)")
+    (add_net "Net-(U6-Pad8)")
+    (add_net "Net-(U6-Pad9)")
+    (add_net "Net-(U7-Pad10)")
+    (add_net "Net-(U7-Pad7)")
+    (add_net "Net-(U7-Pad8)")
+    (add_net "Net-(U7-Pad9)")
     (add_net SCL)
     (add_net SDA)
@@
       (effects (font (size 1 1) (thickness 0.15)))
     )
-    (fp_text value SV2 (at 0 11.6) (layer F.Fab)
+    (fp_text value SV4 (at 0.562 -5.291) (layer F.SilkS)
       (effects (font (size 1 1) (thickness 0.15)))
     )
@@
       (effects (font (size 1 1) (thickness 0.15)))
     )
-    (fp_text value BUZZER_M (at -2.727 2.48776 180) (layer F.SilkS)
+    (fp_text value BUZZER (at -2.727 2.48776 180) (layer F.SilkS)
       (effects (font (size 1 1) (thickness 0.15)))
     )
@@
     (descr "Resistor, Axial_DIN0207 series, Axial, Horizontal, pin pitch=10.16mm, 0.25W = 1/4W, length*diameter=6.3*2.5mm^2, http://cdn-reichelt.de/documents/datenblatt/B400/1_4W%23YAG.pdf")
     (tags "Resistor Axial_DIN0207 series Axial Horizontal pin pitch 10.16mm 0.25W = 1/4W length 6.3mm diameter 2.5mm")
-    (fp_text reference R13 (at 11.83968 -1.49028 180) (layer F.SilkS)
+    (fp_text reference R13 (at 9.55 -2.8 180) (layer F.SilkS)
       (effects (font (size 1 1) (thickness 0.15)))
     )
@@
       (effects (font (size 1 1) (thickness 0.15)))
     )
-    (fp_text value +12V (at -5.14012 -1.12892) (layer F.SilkS)
+    (fp_text value +12V (at 1.55 -3.1) (layer F.SilkS)
       (effects (font (size 1 1) (thickness 0.15)))
     )
@@
     )
   )
+  (gr_text PRESS_INT (at 189.507854 110.569383) (layer F.SilkS)
+    (effects (font (size 1.5 1.5) (thickness 0.3)))
+  )
+  (gr_text PRESSEXT (at 188.357854 55.019383) (layer F.SilkS)
+    (effects (font (size 1.5 1.5) (thickness 0.3)))
+  )
+  (gr_text "FLOW\n" (at 190.707854 78.969383) (layer F.SilkS)
+    (effects (font (size 1.5 1.5) (thickness 0.3)))
+  )
+  (gr_text "FLOW\n" (at 190.907854 103.019383) (layer F.SilkS)
+    (effects (font (size 1.5 1.5) (thickness 0.3)))
+  )
   (gr_text + (at 161.789894 79.478383) (layer F.SilkS)
