File: Doc/PCB/Main_Board_v1_1_SMD/Main_Board_v1_1_smd.kicad_pcb (KiCad board)
At the start: 2 copper layers, 138 x 98 mm, 135 parts, among them J1 SV1, J11 UART_C, J12 I2C Interface LCD_C, J13 BUZZER_C, J2 12V, J24 Conn_01x08, J25 POWEROFF, J27 SV2, J3 UART_M, J4 Conn_01x08, J5 BUZZER_M, J6 I2C Interface LCD_M, J7 TE_3.5mm_Screwless_P2, J8 SV2, J9 SV3, Q1 FDT1600N10ALZ, Q2 FDT1600N10ALZ, Q3 FDT1600N10ALZ, Q4 BSR19A, Q5 BSR19A, Q6 FDT1600N10ALZ, SW1 MUTE, SW10 BREATH, SW11 EP, SW12 +, SW2 HIST, SW3 VOL_MIN, SW4 VOL, SW5 BPM, SW6 IP, SW7 -, SW8 VOL_MAX, SW9 PMAX, U1 LM358, U2 LM78M05_TO252, U3 XPRESS-40, U4 LM78M05_TO252, U5 XPRESS-40, U6 LCD, U7 LCD

Commit message: Fixed bug in Alarm Very High Pressure. Clean up static definition of variables
Parts:
- added FIDUCIAL_TEST_PCB_1C: VAL**, Ventilator:FIDUCIAL_TEST_PCB_1C, F.Cu at (148.4, 36.9)
- added FIDUCIAL_TEST_PCB_1C: VAL**, Ventilator:FIDUCIAL_TEST_PCB_1C, F.Cu at (149.4, 123.9)
- added FIDUCIAL_TEST_PCB_1C: VAL**, Ventilator:FIDUCIAL_TEST_PCB_1C, F.Cu at (44.4, 116.9)
- added FIDUCIAL_TEST_PCB_1C: VAL**, Ventilator:FIDUCIAL_TEST_PCB_1C, F.Cu at (35.4, 36.9)
Changed lines of the file:
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@@
     (tracks 1714)
     (zones 0)
-    (modules 135)
+    (modules 139)
     (nets 88)
   )
@@
   )
   (setup
-    (last_trace_width 0.2)
+    (last_trace_width 0.35)
     (user_trace_width 0.2)
     (user_trace_width 0.35)
@@
     (add_net "Net-(C6-Pad2)")
   )
+  (module Ventilator:FIDUCIAL_TEST_PCB_1C (layer F.Cu)
+    (at 148.357854 36.869383)
+    (fp_text reference FIDUCIAL_TEST_PCB_1C (at 0.1778 -2.286) (layer F.SilkS) hide
+      (effects (font (size 1 1) (thickness 0.15)))
+    )
+    (fp_text value VAL** (at -0.0508 2.413) (layer F.SilkS) hide
+      (effects (font (size 1 1) (thickness 0.15)))
+    )
+    (pad 1 smd circle (at 0 0) (size 1 1) (layers B.Cu B.Mask)
+      (solder_mask_margin 0.75) (clearance 0.75) (zone_connect 0))
+  )
+  (module Ventilator:FIDUCIAL_TEST_PCB_1C (layer F.Cu)
+    (at 149.357854 123.869383)
+    (fp_text reference FIDUCIAL_TEST_PCB_1C (at 0.1778 -2.286) (layer F.SilkS) hide
+      (effects (font (size 1 1) (thickness 0.15)))
+    )
+    (fp_text value VAL** (at -0.0508 2.413) (layer F.SilkS) hide
+      (effects (font (size 1 1) (thickness 0.15)))
+    )
+    (pad 1 smd circle (at 0 0) (size 1 1) (layers B.Cu B.Mask)
+      (solder_mask_margin 0.75) (clearance 0.75) (zone_connect 0))
+  )
+  (module Ventilator:FIDUCIAL_TEST_PCB_1C (layer F.Cu)
+    (at 44.357854 116.869383)
+    (fp_text reference FIDUCIAL_TEST_PCB_1C (at 0.1778 -2.286) (layer F.SilkS) hide
+      (effects (font (size 1 1) (thickness 0.15)))
+    )
+    (fp_text value VAL** (at -0.0508 2.413) (layer F.SilkS) hide
+      (effects (font (size 1 1) (thickness 0.15)))
+    )
+    (pad 1 smd circle (at 0 0) (size 1 1) (layers B.Cu B.Mask)
+      (solder_mask_margin 0.75) (clearance 0.75) (zone_connect 0))
+  )
+  (module Ventilator:FIDUCIAL_TEST_PCB_1C (layer F.Cu)
+    (at 35.357854 36.869383)
+    (fp_text reference FIDUCIAL_TEST_PCB_1C (at 0.1778 -2.286) (layer F.SilkS) hide
+      (effects (font (size 1 1) (thickness 0.15)))
+    )
+    (fp_text value VAL** (at -0.0508 2.413) (layer F.SilkS) hide
+      (effects (font (size 1 1) (thickness 0.15)))
+    )
+    (pad 1 smd circle (at 0 0) (size 1 1) (layers B.Cu B.Mask)
+      (solder_mask_margin 0.75) (clearance 0.75) (zone_connect 0))
+  )
   (module Ventilator:LCD_2x16 locked (layer F.Cu)
     (at 118.857854 85.369383)
@@
       (effects (font (size 1 1) (thickness 0.15)) (justify mirror))
     )
+    (fp_circle (center 3.25 -2.25) (end 1.25 -2.5) (layer B.Fab) (width 0.1))
+    (fp_line (start 6.75 -3) (end 6.75 -1.5) (layer B.SilkS) (width 0.12))
+    (fp_line (start 5.5 1) (end 1 1) (layer B.SilkS) (width 0.12))
+    (fp_line (start -0.25 -1.5) (end -0.25 -3) (layer B.SilkS) (width 0.12))
+    (fp_line (start 1 -5.5) (end 5.5 -5.5) (layer B.SilkS) (width 0.12))
+    (fp_line (start 8 1.25) (end 8 -5.75) (layer B.CrtYd) (width 0.05))
+    (fp_line (start 7.75 -6) (end -1.25 -6) (layer B.CrtYd) (width 0.05))
+    (fp_line (start -1.5 -5.75) (end -1.5 1.25) (layer B.CrtYd) (width 0.05))
+    (fp_line (start -1.25 1.5) (end 7.75 1.5) (layer B.CrtYd) (width 0.05))
+    (fp_line (start -1.5 -6) (end -1.25 -6) (layer B.CrtYd) (width 0.05))
+    (fp_line (start -1.5 -5.75) (end -1.5 -6) (layer B.CrtYd) (width 0.05))
+    (fp_line (start -1.5 1.5) (end -1.25 1.5) (layer B.CrtYd) (width 0.05))
+    (fp_line (start -1.5 1.25) (end -1.5 1.5) (layer B.CrtYd) (width 0.05))
+    (fp_line (start 8 1.5) (end 8 1.25) (layer B.CrtYd) (width 0.05))
+    (fp_line (start 7.75 1.5) (end 8 1.5) (layer B.CrtYd) (width 0.05))
+    (fp_line (start 8 -6) (end 8 -5.75) (layer B.CrtYd) (width 0.05))
+    (fp_line (start 7.75 -6) (end 8 -6) (layer B.CrtYd) (width 0.05))
+    (fp_line (start 0.25 0.75) (end 3.25 0.75) (layer B.Fab) (width 0.1))
+    (fp_line (start 0.25 -5.25) (end 0.25 0.75) (layer B.Fab) (width 0.1))
+    (fp_line (start 6.25 -5.25) (end 0.25 -5.25) (layer B.Fab) (width 0.1))
+    (fp_line (start 6.25 0.75) (end 6.25 -5.25) (layer B.Fab) (width 0.1))
+    (fp_line (start 3.25 0.75) (end 6.25 0.75) (layer B.Fab) (width 0.1))
     (fp_text user %R (at 3.25 -2.25 180) (layer B.Fab)
       (effects (font (size 1 1) (thickness 0.15)) (justify mirror))
     )
-    (fp_line (start 3.25 0.75) (end 6.25 0.75) (layer B.Fab) (width 0.1))
-    (fp_line (start 6.25 0.75) (end 6.25 -5.25) (layer B.Fab) (width 0.1))
-    (fp_line (start 6.25 -5.25) (end 0.25 -5.25) (layer B.Fab) (width 0.1))
-    (fp_line (start 0.25 -5.25) (end 0.25 0.75) (layer B.Fab) (width 0.1))
-    (fp_line (start 0.25 0.75) (end 3.25 0.75) (layer B.Fab) (width 0.1))
-    (fp_line (start 7.75 -6) (end 8 -6) (layer B.CrtYd) (width 0.05))
-    (fp_line (start 8 -6) (end 8 -5.75) (layer B.CrtYd) (width 0.05))
-    (fp_line (start 7.75 1.5) (end 8 1.5) (layer B.CrtYd) (width 0.05))
-    (fp_line (start 8 1.5) (end 8 1.25) (layer B.CrtYd) (width 0.05))
-    (fp_line (start -1.5 1.25) (end -1.5 1.5) (layer B.CrtYd) (width 0.05))
-    (fp_line (start -1.5 1.5) (end -1.25 1.5) (layer B.CrtYd) (width 0.05))
-    (fp_line (start -1.5 -5.75) (end -1.5 -6) (layer B.CrtYd) (width 0.05))
-    (fp_line (start -1.5 -6) (end -1.25 -6) (layer B.CrtYd) (width 0.05))
-    (fp_line (start -1.25 1.5) (end 7.75 1.5) (layer B.CrtYd) (width 0.05))
-    (fp_line (start -1.5 -5.75) (end -1.5 1.25) (layer B.CrtYd) (width 0.05))
-    (fp_line (start 7.75 -6) (end -1.25 -6) (layer B.CrtYd) (width 0.05))
-    (fp_line (start 8 1.25) (end 8 -5.75) (layer B.CrtYd) (width 0.05))
-    (fp_line (start 1 -5.5) (end 5.5 -5.5) (layer B.SilkS) (width 0.12))
-    (fp_line (start -0.25 -1.5) (end -0.25 -3) (layer B.SilkS) (width 0.12))
-    (fp_line (start 5.5 1) (end 1 1) (layer B.SilkS) (width 0.12))
-    (fp_line (start 6.75 -3) (end 6.75 -1.5) (layer B.SilkS) (width 0.12))
-    (fp_circle (center 3.25 -2.25) (end 1.25 -2.5) (layer B.Fab) (width 0.1))
-    (pad 2 thru_hole circle (at 0 -4.5 90) (size 2 2) (drill 1.1) (layers *.Cu *.Mask)
+    (pad 1 thru_hole circle (at 6.5 0 90) (size 2 2) (drill 1.1) (layers *.Cu *.Mask)
+      (net 85 "Net-(R32-Pad2)"))
+    (pad 2 thru_hole circle (at 6.5 -4.5 90) (size 2 2) (drill 1.1) (layers *.Cu *.Mask)
       (net 1 GND))
     (pad 1 thru_hole circle (at 0 0 90) (size 2 2) (drill 1.1) (layers *.Cu *.Mask)
       (net 85 "Net-(R32-Pad2)"))
-    (pad 2 thru_hole circle (at 6.5 -4.5 90) (size 2 2) (drill 1.1) (layers *.Cu *.Mask)
-      (net 1 GND))
-    (pad 1 thru_hole circle (at 6.5 0 90) (size 2 2) (drill 1.1) (layers *.Cu *.Mask)
-      (net 85 "Net-(R32-Pad2)"))
+    (pad 2 thru_hole circle (at 0 -4.5 90) (size 2 2) (drill 1.1) (layers *.Cu *.Mask)
+      (net 1 GND))
     (model ${KISYS3DMOD}/Button_Switch_THT.3dshapes/SW_PUSH_6mm_H13mm.wrl
       (at (xyz 0 0 0))
@@
     (pad "" smd roundrect (at -0.6 -0.825) (size 0.97 1.33) (layers F.Paste) (roundrect_rratio 0.25))
     (pad 9 smd roundrect (at 0 0) (size 2.41 3.3) (layers F.Cu F.Mask) (roundrect_rratio 0.103734))
-    (model ${KISYS3DMOD}/Package_SO.3dshapes/SOIC-8_3.9x4.9mm_P1.27mm.wrl
-      (at (xyz 0 0 0))
-      (scale (xyz 1 1 1))
+    (model ${KISYS3DMOD}/Package_SO.3dshapes/SOIC-8-1EP_3.9x4.9mm_P1.27mm_EP2.41x3.3mm.wrl
+      (at (xyz 0 0 0))
+      (scale (xyz 1 1 1))
